Commit message: Add build logs and error messages for manipulator_control, manipulator_description, and manipulator_moveit_config
- Created command, stderr, stdout, stdout_stderr, and streams logs for manipulator_control, manipulator_description, and manipulator_moveit_config.
- Captured CMake errors related to missing ament_cmake package configuration files.
- Included detailed output of the build process to aid in debugging.

File: ros2_ws/src/manipulator_description/urdf/gripper.xacro (robot description, xacro)
@@ -29,5 +29,5 @@
       <parent link="gripper_base_link"/>
       <child link="left_finger_link"/>
-      <origin xyz="0 0.025 0.03" rpy="0 0 0"/>
+      <origin xyz="0 0.018 0.03" rpy="0 0 0"/>
       <axis xyz="0 1 0"/>
       <limit lower="0.0" upper="0.03" effort="20.0" velocity="0.05"/>
@@ -54,5 +54,5 @@
       <parent link="gripper_base_link"/>
       <child link="right_finger_link"/>
-      <origin xyz="0 -0.025 0.03" rpy="0 0 0"/>
+      <origin xyz="0 -0.018 0.03" rpy="0 0 0"/>
       <axis xyz="0 -1 0"/>
       <limit lower="0.0" upper="0.03" effort="20.0" velocity="0.05"/>
